File: bm1366-1.kicad_sch (KiCad schematic)
At the start: 55 parts, among them U1 25MHz, U10 SGM2036-0v8, U11 SGM2036-1v8, U14 BM1366_mode1

Commit message: Issues about the RI pull-up resistor at the end of the chip chain being fixed
Parts:
- renumbered C2 to C45, C3 to C46, C4 to C47, C5 to C48, C6 to C49, C8 to C50, C8 to C51, C8 to C52, C24 to C53, C24 to C54, C14 to C55, C12 to C56, C15 to C57, C16 to C58, C17 to C59, C8 to C60, C18 to C61, C8 to C62, C10 to C63, C2 to C64, C11 to C65, C3 to C66, C4 to C67, C13 to C68, C6 to C69, C5 to C70, C8 to C71, C12 to C72, C8 to C73, C14 to C74, C15 to C75, C16 to C76, C17 to C77, C18 to C78, R6 to R28, R6 to R33, TP13 to TP33, TP13 to TP34, TP13 to TP35, TP13 to TP36, TP13 to TP37, TP13 to TP38, TP13 to TP39, TP13 to TP40, TP13 to TP41, U14 to U12, U14 to U13, U1 to U14
