File: bm1366-2.kicad_sch (KiCad schematic)
At the start: 74 parts, among them U1 25MHz, U15 TLV3544, U16 SGM2036-1v8, U17 SGM2036-0v8, U18 BM1366_mode0, U20 BM1366_mode0

Commit message: Issues about the RI pull-up resistor at the end of the chip chain being fixed
Parts:
- renumbered C3 to C100, C13 to C101, C4 to C102, C6 to C103, C5 to C104, C8 to C105, C8 to C106, C12 to C107, C15 to C108, C17 to C109, C14 to C110, C8 to C111, C8 to C112, C16 to C113, C18 to C114, C2 to C79, C3 to C80, C4 to C81, C8 to C82, C5 to C83, C8 to C84, C6 to C85, C8 to C86, C24 to C87, C24 to C88, C14 to C89, C12 to C90, C15 to C91, C14 to C92, C8 to C93, C17 to C94, C8 to C95, C18 to C96, C10 to C97, C2 to C98, C11 to C99, R6 to R34, R6 to R35, R6 to R36, R6 to R37, R6 to R42, R6 to R43, R6 to R44, R6 to R45, R6 to R46, R6 to R47, R6 to R48, R6 to R49, R6 to R50, R6 to R51, R6 to R52, R6 to R53, R6 to R54, R6 to R55, TP13 to TP42, TP13 to TP43, TP13 to TP44, TP13 to TP45, TP13 to TP46, TP13 to TP47, TP13 to TP48, TP13 to TP49, TP13 to TP50, U1 to U19
