File: bm1366-3.kicad_sch (KiCad schematic)
At the start: 79 parts, among them U1 25MHz, U14 BM1366_mode1, U21 TLV3544, U23 SGM2036-0v8, U24 SGM2036-1v8

Commit message: Issues about the RI pull-up resistor at the end of the chip chain being fixed
Parts:
- added R80: 10k, Resistor_SMD:R_0402_1005Metric, symbol Device:R_US
- renumbered C2 to C115, C3 to C116, C4 to C117, C5 to C118, C6 to C119, C8 to C120, C8 to C121, C8 to C122, C14 to C123, C12 to C124, C24 to C125, C24 to C126, C15 to C127, C16 to C128, C17 to C129, C8 to C130, C18 to C131, C8 to C132, C2 to C133, C10 to C134, C3 to C135, C4 to C136, C11 to C137, C6 to C138, C5 to C139, C13 to C140, C8 to C141, C8 to C142, C12 to C143, C15 to C144, C17 to C145, C14 to C146, C8 to C147, C8 to C148, C16 to C149, C18 to C150, R6 to R56, R6 to R57, R6 to R58, R6 to R59, R6 to R60, R6 to R61, R6 to R62, R6 to R67, R6 to R68, R6 to R69, R6 to R70, R6 to R71, R6 to R72, R6 to R73, R6 to R74, R6 to R75, R6 to R76, R6 to R77, TP13 to TP51, TP13 to TP52, TP13 to TP53, TP13 to TP54, TP13 to TP55, TP13 to TP56, TP13 to TP57, TP13 to TP58, TP13 to TP59, TP13 to TP60, TP13 to TP61, TP13 to TP62, TP13 to TP63, U14 to U22, U14 to U25, U1 to U26
Connections:
- net 1V8: now also R80.2
- net RI3: now also R80.1
Other:
- moved on the sheet: TP61
