File: esp32.kicad_sch (KiCad schematic)
At the start: 53 parts, among them J4 TC2030-IDC, J5 Conn_01x04, J6 Conn_01x06, J8 USB_C_Receptacle_USB2.0, SW1 SWITCH-SPST, SW2 SWITCH-SPST, U5 SN74AVC4T774, U6 ESP32-S3-WROOM-1, Y1 32.768kHz

Commit message: Issues about the RI pull-up resistor at the end of the chip chain being fixed
Parts:
- renumbered C50 to C32, C25 to C34, C25 to C35, J8 to J7, R20 to R18, R8 to R21, R3 to R22, R5 to R23
