File: fan.kicad_sch (KiCad schematic)
At the start: 16 parts, among them J8 Conn_01x04, J9 Conn_01x04, U7 TMP1075, U8 TMP1075, U9 EMC2302

Commit message: Issues about the RI pull-up resistor at the end of the chip chain being fixed
Parts:
- renumbered R7 to R26, R7 to R27
