File: power.kicad_sch (KiCad schematic)
At the start: 65 parts, among them J3 Conn_02x05_Odd_Even, T1 net-tie, U1 LMR54410, U2 RT9080-33GJ5, U3 TPS546D24ARVFR, U4 MIC5504

Commit message: Issues about the RI pull-up resistor at the end of the chip chain being fixed
Parts:
- renumbered C8 to C12, C8 to C6, R6 to R1, R7 to R17, R6 to R2, R6 to R3
